File: PCBs/sisyphus/sisyphus.kicad_sch (KiCad schematic)
At the start: 75 parts, among them J1 Light sensor, J10 Keyboard, J2 USB_C_Receptacle_USB2.0_14P, J3 AUX USB, J4 USB_BOOT, J5 Speaker, J6 Battery, J7 SWD, J8 Limit SW, J9 RGB_CONN, Q1 AO3401A, Q2 FS8205, SW1 SW_SPDT_321, U1 TPS62293, U2 USBLC6-2P6, U3 BQ25619, U4 W25Q128JVS, U5 MAX98357A, U6 DW01A, U7 RP2040, Y1 ABM8-272-T3

Commit message: Some schematic readability improved. Minor changes in PCB
Parts:
- removed C1: 47nF, Capacitor_SMD:C_0402_1005Metric, symbol Device:C_Small
- removed C10: 10uF, Capacitor_SMD:C_0402_1005Metric, symbol Device:C_Small
- removed C2, C4, C5, C6, C8: 10uF, Capacitor_SMD:C_0402_1005Metric, symbol Device:C
- removed C25, C9: 100nF, Capacitor_SMD:C_0402_1005Metric, symbol Device:C_Small
- removed C3: 1uF, Capacitor_SMD:C_0402_1005Metric, symbol Device:C_Small
- removed C7: 4.7uF, Capacitor_SMD:C_0402_1005Metric, symbol Device:C_Small
- removed D1: D_Schottky, Diode_SMD:D_0402_1005Metric, symbol Device:D_Schottky_Small
- removed D2: LED, LED_SMD:LED_0402_1005Metric, symbol Device:LED
- removed J1: Light sensor, Connector_JST:JST_XH_S5B-XH-A_1x05_P2.50mm_Horizontal, symbol Connector_Generic:Conn_01x05
- removed J10: Keyboard, Connector_JST:JST_XH_S8B-XH-A_1x08_P2.50mm_Horizontal, symbol Connector_Generic:Conn_01x08
- removed J2: USB_C_Receptacle_USB2.0_14P, Connector_USB:USB_C_Receptacle_G-Switch_GT-USB-7010ASV, symbol Connector:USB_C_Receptacle_USB2.0_14P
- removed J3: AUX USB, Connector_PinHeader_2.54mm:PinHeader_1x04_P2.54mm_Vertical, symbol Connector:Conn_01x04_Pin
- removed J5: Speaker, Connector_PinHeader_2.54mm:PinHeader_1x02_P2.54mm_Vertical, symbol Connector_Generic:Conn_01x02
- removed J6: Battery, Connector_JST:JST_PH_S2B-PH-SM4-TB_1x02-1MP_P2.00mm_Horizontal, symbol Connector_Generic:Conn_01x02
- removed J8: Limit SW, Connector_PinSocket_2.54mm:PinSocket_1x02_P2.54mm_Vertical, symbol Connector_Generic:Conn_01x02
- removed J9: RGB_CONN, Connector_PinHeader_2.54mm:PinHeader_1x03_P2.54mm_Vertical, symbol Connector:Conn_01x03_Pin
- removed JP1: Gain select, Jumper:SolderJumper-3_P1.3mm_Open_RoundedPad1.0x1.5mm, symbol Jumper:SolderJumper_3_Open
- removed L1: 1uH, Inductor_SMD:L_0402_1005Metric, symbol Device:L
- removed L2: 2.2uH 1A, Inductor_SMD:L_0603_1608Metric, symbol Device:L
- removed Q1: AO3401A, Package_TO_SOT_SMD:SOT-23, symbol Transistor_FET:AO3401A
- removed Q2: FS8205, Package_TO_SOT_SMD:SOT-23-6, symbol easyeda2kicad:FS8205
- removed R1: 1M, Resistor_SMD:R_0402_1005Metric, symbol Device:R_Small
- removed R10: DNF, Resistor_SMD:R_0402_1005Metric, symbol Device:R_Small
- removed R16: 100, Resistor_SMD:R_0402_1005Metric, symbol Device:R_Small
- removed R17: 1k, Resistor_SMD:R_0402_1005Metric, symbol Device:R_Small
- removed R2, R3: 5.1k, Resistor_SMD:R_0402_1005Metric, symbol Device:R_Small
- removed R4: 220, Resistor_SMD:R_0402_1005Metric, symbol Device:R_Small
- removed R5: 10k, Resistor_SMD:R_0402_1005Metric, symbol Device:R_Small
- removed R6: 5.3k, Resistor_SMD:R_0402_1005Metric, symbol Device:R_Small
- removed R7: 31.14k, Resistor_SMD:R_0402_1005Metric, symbol Device:R_Small
- removed SW1: SW_SPDT_321, Connector_PinHeader_2.54mm:PinHeader_1x03_P2.54mm_Vertical, symbol Switch:SW_SPDT_321
- removed TH1: 10k NTC, Connector_PinHeader_2.54mm:PinHeader_1x02_P2.54mm_Vertical, symbol Device:Thermistor_NTC
- removed U1: TPS62293, Package_SON:WSON-6-1EP_2x2mm_P0.65mm_EP1x1.6mm_ThermalVias, symbol Sisyphus:TPS62293
- removed U2: USBLC6-2P6, Package_TO_SOT_SMD:SOT-666, symbol Power_Protection:USBLC6-2P6
- removed U3: BQ25619, Package_DFN_QFN:Texas_RTW_WQFN-24-1EP_4x4mm_P0.5mm_EP2.7x2.7mm_ThermalVias, symbol Sisyphus:BQ25619
- removed U5: MAX98357A, Package_DFN_QFN:TQFN-16-1EP_3x3mm_P0.5mm_EP1.23x1.23mm, symbol Audio:MAX98357A
- removed U6: DW01A, Package_TO_SOT_SMD:SOT-23-6, symbol Battery_Management:DW01A
- removed U8: ~, Package_DFN_QFN:WQFN-24-1EP_4x4mm_P0.5mm_EP2.45x2.45mm, symbol Sisyphus:TCA8418
Connections:
- net XIN: no longer names the net of C23.1, U7.20 (XIN), Y1.1
- net XOUT: no longer names the net of R15.1, U7.21 (XOUT)
- no-connect marks 3 -> 0
Other:
- added sheet Batery and power (power.kicad_sch)
- added sheet Peripheral (peripheral.kicad_sch)
- note added: "Decoupling for LEDs"
- note added: "Flash Pins"
- note removed: "Battery charger"
- note removed: "Battery connector"
- note removed: "Crystal"
- note removed: "Decoupling for LEDs (and stuff)"
- note removed: "Flash"
- note removed: "GND is 12dB VDD is 6dB"
- note removed: "I2S DAC and amplifier"
- note removed: "Keyboard controller"
- note removed: "Limit switch connector"
- note removed: "Place close to IC"
- note removed: "Place close to battery"
- note removed: "RGBW sensor connector"
- note removed: "RP2040"
- note removed: "Step-down"
- note removed: "USB-C"
- note removed: "WS2812B connector"
- moved on the sheet: C11, C12, C13, C14, C15, C16, C17, C18, C19, C20, C21, C22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
