File: PCBs/sisyphus/sisyphus.kicad_sch (KiCad schematic)
At the start: 66 parts, among them J1 Battery, J2 USB_C_Receptacle_USB2.0_14P, J3 USB_BOOT, J4 SPK, J5 RGB_CONN, J6 AUX, J7 SWD, J8 KEYB, J9 PWR-BTN, Q1 AO3401A, SW1 SW_SPDT_321, U1 TPS62291, U2 MP2667, U3 USBLC6-2P6, U4 MAX17048, U5 W25Q128JVP, U6 TCA8418, U7 MAX98357A, U8 RP2040, Y1 ABM8-272-T3

Commit message: Add GND return paths, move USB_BOOT
Parts:
- J3: footprint Connector_PinHeader_2.54mm:PinHeader_1x02_P2.54mm_Vertical -> Connector_PinHeader_1.00mm:PinHeader_1x02_P1.00mm_Vertical
Changed lines of the file:
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@@
 			)
 		)
-		(property "Footprint" "Connector_PinHeader_2.54mm:PinHeader_1x02_P2.54mm_Vertical"
+		(property "Footprint" "Connector_PinHeader_1.00mm:PinHeader_1x02_P1.00mm_Vertical"
 			(at 27.94 102.87 0)
 			(hide yes)

Commit message: PCB smaller now
Connections:
- net KEYPAD_INT: now also U8.28 (GPIO17); no longer U8.30 (GPIO19)
- net KEYPAD_RESET: now also U8.29 (GPIO18); no longer U8.31 (GPIO20)
- net RGB_DATA: now also U8.30 (GPIO19); no longer U8.6 (GPIO4)
Changed lines of the file:
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@@
 	(wire
 		(pts
-			(xy 227.33 207.01) (xy 242.57 207.01)
+			(xy 227.33 201.93) (xy 242.57 201.93)
 		)
 		(stroke
@@
 	(wire
 		(pts
-			(xy 227.33 209.55) (xy 242.57 209.55)
+			(xy 227.33 204.47) (xy 242.57 204.47)
 		)
 		(stroke
@@
 	(wire
 		(pts
-			(xy 227.33 168.91) (xy 237.49 168.91)
+			(xy 227.33 207.01) (xy 237.49 207.01)
 		)
 		(stroke
@@
 	)
 	(label "RGB_DATA"
-		(at 237.49 168.91 180)
+		(at 237.49 207.01 180)
 		(effects
 			(font
@@
 	)
 	(label "KEYPAD_RESET"
-		(at 242.57 209.55 180)
+		(at 242.57 204.47 180)
 		(effects
 			(font
@@
 	)
 	(label "KEYPAD_INT"
-		(at 242.57 207.01 180)
+		(at 242.57 201.93 180)
 		(effects
 			(font

Commit message: PCB Hopefuly done
Connections:
- net AUX_LED: now also U8.7 (GPIO5); no longer U8.16 (GPIO13)
- net LMT_SW: now also U8.6 (GPIO4); no longer U8.15 (GPIO12)
Changed lines of the file:
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@@
 	(wire
 		(pts
-			(xy 227.33 189.23) (xy 237.49 189.23)
+			(xy 227.33 168.91) (xy 237.49 168.91)
 		)
 		(stroke
@@
 	(wire
 		(pts
-			(xy 227.33 191.77) (xy 237.49 191.77)
+			(xy 227.33 171.45) (xy 237.49 171.45)
 		)
 		(stroke
@@
 	)
 	(label "AUX_LED"
-		(at 237.49 191.77 180)
+		(at 237.49 171.45 180)
 		(effects
 			(font
@@
 	)
 	(label "LMT_SW"
-		(at 237.49 189.23 180)
-		(effects
-			(font
+		(at 237.49 168.91 180)
+		(effects
+			(font
