File: PCBs/sisyphus/peripheral.kicad_sch (KiCad schematic)
At the start: 17 parts, among them J1 Light sensor, J10 Keyboard, J2 USB_C_Receptacle_USB2.0_14P, J3 AUX USB, J5 Speaker, J8 Limit SW, J9 RGB_CONN, U2 USBLC6-2P6, U5 MAX98357A

Commit message: Fix things on PCB, update inductor size
Parts:
- U8: value ~ -> TCA8418
Changed lines of the file:
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@@
 			)
 		)
-		(property "Value" "~"
+		(property "Value" "TCA8418"
 			(at 195.1833 76.2 0)
 			(effects

Commit message: Add the first actually ordered version of the PCB
Parts:
- D2: renamed from D1; value D_Schottky -> D_shottky; footprint Diode_SMD:D_0402_1005Metric -> Diode_SMD:D_SOD-123; LCSC Part (none) -> https://lcsc.com/product-detail/Schottky-Diodes_FUXINSEMI-M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
- J4: renamed from J2; LCSC Part (none) -> https://lcsc.com/product-detail/USB-Connectors_G-Switch-GT-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
- J5: renamed from J10; LCSC Part (none) -> https://lcsc.com/product-detail/Wire-To-Board-Connector_JST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
- J7: renamed from J1; LCSC Part (none) -> https://lcsc.com/product-detail/Wire-To-Board-Connector_JST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
- U5: renamed from U2; LCSC Part (none) -> https://lcsc.com/product-detail/ESD-and-Surge-Protection-TV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
- U6: renamed from U8; LCSC Part (none) -> https://lcsc.com/product-detail/I-O-Expanders_Texas-Instrum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
- U7: renamed from U5; LCSC Part (none) -> https://lcsc.com/product-detail/Audio-Amplifiers_Analog-Dev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
- renumbered C9 to C24, C10 to C25, J5 to J10, J3 to J6, R2 to R12, R3 to R13, R10 to R14
