File: PCBs/sisyphus/power.kicad_sch (KiCad schematic)
At the start: 22 parts, among them J6 Battery, Q1 AO3401A, SW1 SW_SPDT_321, U1 TPS62293, U3 BQ25619

Commit message: Fix things on PCB, update inductor size
Parts:
- removed J6: Battery, Connector_JST:JST_PH_S2B-PH-SM4-TB_1x02-1MP_P2.00mm_Horizontal, symbol Connector_Generic:Conn_01x02
- removed TH1: 10k NTC, Connector_PinHeader_2.54mm:PinHeader_1x02_P2.54mm_Vertical, symbol Device:Thermistor_NTC
- added J6: Battery, Connector_JST:JST_PH_S3B-PH-SM4-TB_1x03-1MP_P2.00mm_Horizontal, symbol Connector_Generic:Conn_01x03
- L1: value 1uH -> 1uH 2A; footprint Inductor_SMD:L_0402_1005Metric -> Inductor_SMD:L_0603_1608Metric
- L2: value 2.2uH 1A -> 2.2uH 1.2A
Connections:
- net +BATT: now also J6.3 (Pin_3)
- net GND: now also J6.1 (Pin_1)
- net NTC: now reaches R6.2, R7.1, U3.11 (TS)
- net NTC: now also J6.2 (Pin_2)
Other:
- note added: "10k NTC on battery"
- note removed: "Place close to battery"
Changed lines of the file:
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@@
 		)
 	)
-	(text "Place close to battery"
+	(text "10k NTC on battery"
 		(exclude_from_sim no)
-		(at 127 134.874 0)
+		(at 109.982 127.254 0)
 		(effects
 			(font
@@
 		(color 0 0 0 0)
 	)
-	(junction
-		(at 97.79 135.89)
-		(diameter 0)
-		(color 0 0 0 0)
-	)
 	(no_connect
 		(at 115.57 68.58)
@@
 	(wire
 		(pts
-			(xy 97.79 133.35) (xy 97.79 135.89)
-		)
-		(stroke
-			(width 0)
-			(type default)
-		)
-	)
-	(wire
-		(pts
-			(xy 97.79 135.89) (xy 97.79 138.43)
+			(xy 97.79 133.35) (xy 97.79 138.43)
 		)
 		(stroke
@@
 	(wire
 		(pts
-			(xy 114.3 135.89) (xy 114.3 134.62)
-		)
-		(stroke
-			(width 0)
-			(type default)
-		)
-	)
-	(wire
-		(pts
 			(xy 57.15 110.49) (xy 57.15 113.03)
 		)
@@
 	(wire
 		(pts
-			(xy 50.8 99.06) (xy 48.26 99.06)
+			(xy 50.8 101.6) (xy 48.26 101.6)
 		)
 		(stroke
@@
 	(wire
 		(pts
-			(xy 114.3 127) (xy 114.3 125.73)
-		)
-		(stroke
-			(width 0)
-			(type default)
-		)
-	)
-	(wire
-		(pts
 			(xy 232.41 86.36) (xy 245.11 86.36)
 		)
@@
 	(wire
 		(pts
-			(xy 63.5 85.09) (xy 68.58 85.09)
+			(xy 48.26 99.06) (xy 50.8 99.06)
 		)
 		(stroke
@@
 	(wire
 		(pts
-			(xy 127 73.66) (xy 127 74.93)
+			(xy 63.5 85.09) (xy 68.58 85.09)
 		)
 		(stroke
@@
 	(wire
 		(pts
-			(xy 194.31 101.6) (xy 194.31 99.06)
+			(xy 127 73.66) (xy 127 74.93)
 		)
 		(stroke
@@
 	(wire
 		(pts
-			(xy 125.73 110.49) (xy 125.73 107.95)
+			(xy 194.31 101.6) (xy 194.31 99.06)
 		)
 		(stroke
@@
 	(wire
 		(pts
-			(xy 97.79 115.57) (xy 97.79 118.11)
+			(xy 125.73 110.49) (xy 125.73 107.95)
 		)
 		(stroke
@@
 	(wire
 		(pts
-			(xy 237.49 83.82) (xy 229.87 83.82)
+			(xy 97.79 115.57) (xy 97.79 118.11)
 		)
 		(stroke
@@
 	(wire
 		(pts
-			(xy 107.95 82.55) (xy 113.03 82.55)
+			(xy 237.49 83.82) (xy 229.87 83.82)
 		)
 		(stroke
@@
 	(wire
 		(pts
-			(xy 97.79 82.55) (xy 97.79 83.82)
+			(xy 107.95 82.55) (xy 113.03 82.55)
 		)
 		(stroke
@@
 	(wire
 		(pts
-			(xy 97.79 135.89) (xy 114.3 135.89)
+			(xy 97.79 82.55) (xy 97.79 83.82)
 		)
 		(stroke
@@
 		)
 	)
+	(label "NTC"
+		(at 114.3 125.73 180)
+		(effects
+			(font
+				(size 1.27 1.27)
+			)
+			(justify right bottom)
+		)
+	)
 	(label "SW"
 		(at 95.25 82.55 0)
@@
 		)
 	)
+	(label "NTC"
+		(at 50.8 99.06 0)
+		(effects
+			(font
+				(size 1.27 1.27)
+			)
+			(justify left bottom)
+		)
+	)
 	(global_label "PMIC_INT"
 		(shape input)
@@
 	)
 	(symbol
-		(lib_id "Device:Thermistor_NTC")
-		(at 114.3 130.81 0)
-		(unit 1)
-		(exclude_from_sim no)
-		(in_bom no)
-		(on_board yes)
-		(dnp no)
-		(fields_autoplaced yes)
-		(property "Reference" "TH1"
-			(at 116.84 129.8574 0)
-			(effects
-				(font
-					(size 1.27 1.27)
-				)
-				(justify left)
-			)
-		)
-		(property "Value" "10k NTC"
-			(at 116.84 132.3974 0)
-			(effects
-				(font
-					(size 1.27 1.27)
-				)
-				(justify left)
-			)
-		)
-		(property "Footprint" "Connector_PinHeader_2.54mm:PinHeader_1x02_P2.54mm_Vertical"
-			(at 114.3 129.54 0)
-			(effects
-				(font
-					(size 1.27 1.27)
-				)
-				(hide yes)
-			)
-		)
-		(property "Datasheet" "~"
-			(at 114.3 129.54 0)
-			(effects
-				(font
-					(size 1.27 1.27)
-				)
-				(hide yes)
-			)
-		)
-		(property "Description" "Temperature dependent resistor, negative temperature coefficient"
-			(at 114.3 130.81 0)
-			(effects
-				(font
-					(size 1.27 1.27)
-				)
-				(hide yes)
-			)
-		)
-		(pin "2"
-		)
-		(pin "1"
-		)
-		(instances
-			(project "sisyphus"
-				(path "/8c0b3d8b-46d3-4173-ab1e-a61765f77d61/129d5b5c-8633-4296-9137-1037c935b2ab"
-					(reference "TH1")
-					(unit 1)
-				)
-			)
-		)
-	)
-	(symbol
 		(lib_id "Device:C")
 		(at 135.89 115.57 0)
@@
 	)
 	(symbol
-		(lib_id "Connector_Generic:Conn_01x02")
-		(at 43.18 99.06 180)
+		(lib_id "power:+3V3")
+		(at 194.31 76.2 0)
 		(unit 1)
 		(exclude_from_sim no)
@@
 		(on_board yes)
 		(dnp no)
-		(fields_autoplaced yes)
-		(property "Reference" "J6"
-			(at 43.18 90.17 0)
+		(property "Reference" "#PWR06"
+			(at 194.31 80.01 0)
 			(effects
 				(font
 					(size 1.27 1.27)
 				)
+				(hide yes)
 			)
 		)
-		(property "Value" "Battery"
-			(at 43.18 92.71 0)
+		(property "Value" "+3V3"
+			(at 194.691 71.8058 0)
 			(effects
 				(font
@@
 			)
 		)
-		(property "Footprint" "Connector_JST:JST_PH_S2B-PH-SM4-TB_1x02-1MP_P2.00mm_Horizontal"
-			(at 43.18 99.06 0)
+		(property "Footprint" ""
+			(at 194.31 76.2 0)
 			(effects
 				(font
@@
 			)
 		)
-		(property "Datasheet" "~"
-			(at 43.18 99.06 0)
+		(property "Datasheet" ""
+			(at 194.31 76.2 0)
 			(effects
 				(font
@@
 			)
 		)
-		(property "Description" "Generic connector, single row, 01x02, script generated (kicad-library-utils/schlib/autogen/connector/)"
-			(at 43.18 99.06 0)
+		(property "Description" ""
+			(at 194.31 76.2 0)
 			(effects
 				(font
 					(size 1.27 1.27)
 				)
-				(hide yes)
 			)
 		)
 		(pin "1"
 		)
-		(pin "2"
-		)
 		(instances
 			(project "sisyphus"
 				(path "/8c0b3d8b-46d3-4173-ab1e-a61765f77d61/129d5b5c-8633-4296-9137-1037c935b2ab"
-					(reference "J6")
+					(reference "#PWR06")
 					(unit 1)
 				)
@@
 	)
 	(symbol
-		(lib_id "power:+3V3")
-		(at 194.31 76.2 0)
+		(lib_id "Connector_Generic:Conn_01x03")
+		(at 43.18 99.06 180)
 		(unit 1)
 		(exclude_from_sim no)
@@
 		(on_board yes)
 		(dnp no)
-		(property "Reference" "#PWR06"
-			(at 194.31 80.01 0)
+		(fields_autoplaced yes)
+		(property "Reference" "J6"
+			(at 43.18 90.17 0)
 			(effects
 				(font
 					(size 1.27 1.27)
 				)
-				(hide yes)
 			)
 		)
-		(property "Value" "+3V3"
-			(at 194.691 71.8058 0)
+		(property "Value" "Battery"
+			(at 43.18 92.71 0)
 			(effects
 				(font
@@
 			)
 		)
-		(property "Footprint" ""
-			(at 194.31 76.2 0)
+		(property "Footprint" "Connector_JST:JST_PH_S3B-PH-SM4-TB_1x03-1MP_P2.00mm_Horizontal"
+			(at 43.18 99.06 0)
 			(effects
 				(font
@@
 			)
 		)
-		(property "Datasheet" ""
-			(at 194.31 76.2 0)
+		(property "Datasheet" "~"
+			(at 43.18 99.06 0)
 			(effects
 				(font
@@
 			)
 		)
-		(property "Description" ""
-			(at 194.31 76.2 0)
+		(property "Description" "Generic connector, single row, 01x03, script generated (kicad-library-utils/schlib/autogen/connector/)"
+			(at 43.18 99.06 0)
 			(effects
 				(font
 					(size 1.27 1.27)
 				)
+				(hide yes)
 			)
 		)
+		(pin "3"
+		)
+		(pin "2"
+		)
 		(pin "1"
 		)
 		(instances
-			(project "sisyphus"
+			(project ""
 				(path "/8c0b3d8b-46d3-4173-ab1e-a61765f77d61/129d5b5c-8633-4296-9137-1037c935b2ab"
-					(reference "#PWR06")
+					(reference "J6")
 					(unit 1)
 				)
@@
 	(symbol
 		(lib_id "power:GND")
-		(at 50.8 99.06 0)
+		(at 50.8 101.6 0)
 		(unit 1)
 		(exclude_from_sim no)
@@
 		(fields_autoplaced yes)
 		(property "Reference" "#PWR053"
-			(at 50.8 105.41 0)
+			(at 50.8 107.95 0)
 			(effects
 				(font
@@
 		)
 		(property "Value" "GND"
-			(at 50.8 104.14 0)
+			(at 50.8 106.68 0)
 			(effects
 				(font
@@
 		)
 		(property "Footprint" ""
-			(at 50.8 99.06 0)
+			(at 50.8 101.6 0)
 			(effects
 				(font
@@
 		)
 		(property "Datasheet" ""
-			(at 50.8 99.06 0)
+			(at 50.8 101.6 0)
 			(effects
 				(font
@@
 		)
 		(property "Description" "Power symbol creates a global label with name \"GND\" , ground"
-			(at 50.8 99.06 0)
+			(at 50.8 101.6 0)
 			(effects
 				(font
@@
 			)
 		)
-		(property "Value" "1uH"
+		(property "Value" "1uH 2A"
 			(at 102.87 80.01 90)
 			(effects
@@
 			)
 		)
-		(property "Footprint" "Inductor_SMD:L_0402_1005Metric"
+		(property "Footprint" "Inductor_SMD:L_0603_1608Metric"
 			(at 102.87 82.55 0)
 			(effects
@@
 			)
 		)
-		(property "Value" "2.2uH 1A"
+		(property "Value" "2.2uH 1.2A"
 			(at 200.66 81.28 90)
 			(effects

Commit message: Add the first actually ordered version of the PCB
Parts:
- removed R7: 31.14k, Resistor_SMD:R_0402_1005Metric, symbol Device:R_Small
- C16: renamed from C1; LCSC Part (none) -> https://lcsc.com/product-detail/Multilayer-Ceramic-Capacito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
- D1: renamed from D2; footprint LED_SMD:LED_0402_1005Metric -> LED_SMD:LED_0603_1608Metric
- J3: renamed from J6; LCSC Part (none) -> https://lcsc.com/product-detail/Wire-To-Board-Connector_JST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
- L1: LCSC Part (none) -> https://lcsc.com/product-detail/Inductors-SMD_Murata-Electr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
- L2: footprint Inductor_SMD:L_0603_1608Metric -> Inductor_SMD:L_0805_2012Metric
- Q1: LCSC Part (none) -> https://lcsc.com/product-detail/MOSFETs_UMW-Youtai-Semicond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
- R11: renamed from R6; value 5.3k -> 10k
- R9: renamed from R4; value 220 -> 330
- U3: renamed from U1; value TPS62293 -> TPS62291; LCSC Part (none) -> https://lcsc.com/product-detail/DC-DC-Converters_Texas-Inst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
- U4: renamed from U3; LCSC Part (none) -> https://lcsc.com/product-detail/Battery-Management_Texas-In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
- renumbered C2 to C17, C3 to C18, C4 to C19, C5 to C20, C6 to C21, C7 to C22, C8 to C23, R5 to R10, R1 to R8
