File: PCBs/rgb_sensor/rgb_sensor.kicad_sch (KiCad schematic)
At the start: 10 parts, among them J1 Conn_01x05, Q1 AO3401A, U1 VEML3328

Commit message: Update RGB sensor PCB
Redesign for a JST SH connector so it actually fits in the bezel of the keyboard matrix
Parts:
- J1: footprint Connector_JST:JST_XH_S5B-XH-A_1x05_P2.50mm_Horizontal -> Connector_JST:JST_SH_SM05B-SRSS-TB_1x05-1MP_P1.00mm_Horizontal
Changed lines of the file:
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@@
 			)
 		)
-		(property "Footprint" "Connector_JST:JST_XH_S5B-XH-A_1x05_P2.50mm_Horizontal"
+		(property "Footprint" "Connector_JST:JST_SH_SM05B-SRSS-TB_1x05-1MP_P1.00mm_Horizontal"
 			(at 99.06 93.98 0)
 			(effects
