File: PCBs/rgb_sensor/rgb_sensor.kicad_sch (KiCad schematic)
At the start: 10 parts, among them J1 Conn_01x05, Q1 AO3401A, U1 VEML3328

Commit message: Initial changes for Gamma RGB sensor board
Parts:
- removed J1: Conn_01x05, Connector_JST:JST_SH_SM05B-SRSS-TB_1x05-1MP_P1.00mm_Horizontal, symbol Connector_Generic:Conn_01x05
- added C2: 100n, Capacitor_SMD:C_0402_1005Metric, symbol Device:C_Small
- added J1: Conn_01x06_MountingPin, Connector_JST:JST_SH_SM06B-SRSS-TB_1x06-1MP_P1.00mm_Horizontal, symbol Connector_Generic_MountingPin:Conn_01x06_MountingPin
- added U2: TMAG5273A1QDBVR, rgb_sensor:DBV0006A-MFG, symbol sisyphus:TMAG5273A1QDBVR
Connections:
- net +3V3: now also C2.1, J1.6 (Pin_6), U2.4 (VCC)
- net AUX_LED: now also J1.5 (Pin_5)
- net GND: now also C2.2, J1.1 (Pin_1), J1.MP (MountPin), U2.2 (TEST), U2.3 (GND)
- net SCL: now also J1.4 (Pin_4), U2.1 (SCL)
- net SDA: now also J1.3 (Pin_3), U2.6 (SDA)
- new net INT_HALL: J1.2 (Pin_2), U2.5 (INT_N)
